File: ecksdee-wifi-card-rounded.kicad_pcb (KiCad board)
At the start: 2 copper layers, 120 x 72.7 mm, 37 parts, among them IC1 SN74HC688PWR, IC2 ESP-07S, IC3 TL16C550CPTR, J1 Bus_ISA_8bit, J2 TYPE-C-31-M-12, J3 95278-101A04LF, J4 95278-801A08LF, J5 Conn_01x04, Q1 UMH3N, U1 AMS1117-3.3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

Commit message: Initial Commit
Parts:
- removed C10: 0.1uF, Capacitor_SMD:C_0402_1005Metric
- moved R2 1.18 mm to (179.4, 82.4), turned to 135 degrees
- moved R4 0.80 mm to (176.8, 84.7), turned to 135 degrees
Connections:
- J2 pad B6: unconnected-(J2-PadB6) -> /USB_D+
- J2 pad B7: unconnected-(J2-PadB7) -> /USB_D-
- U2 pad 10: Net-(U2-Pad10) -> unconnected-(U2-Pad10)
Routing:
- net /USB_D-: track 8.37 -> 15.1 mm, vias 0 -> 2
- net /USB_D+: track 8.32 -> 11.0 mm
- net VCC: track 221.2 -> 223.5 mm, vias 9 -> 10
- net Net-(U2-Pad10): track 1.56 -> 0.00 mm
Other:
- board text added: "5V RX RX GND"
- board text removed: "5V TX RX GND"
- board text removed: "REV 2"
